Commit message: Add CAD files sim

File: feely_drone_common/assets/gripper.urdf (robot description, URDF)
Before this commit: robot gripper, 17 links, 16 joints
Links:
- link arm1_link1: geometry collision cylinder length=0.15 radius=0.01; visual mesh filename=./meshes/ProximalPhalang.dae
- link arm1_link2: geometry collision cylinder length=0.25 radius=0.01; visual mesh filename=./meshes/MiddlePhalang.dae
- link arm1_link3: geometry collision cylinder length=0.25 radius=0.01; visual mesh filename=./meshes/DistalPhalang.dae
- link arm2_link1: geometry collision cylinder length=0.15 radius=0.01; visual mesh filename=./meshes/ProximalPhalang.dae
- link arm2_link2: geometry collision cylinder length=0.25 radius=0.01; visual mesh filename=./meshes/MiddlePhalang.dae
- link arm2_link3: geometry collision cylinder length=0.25 radius=0.01; visual mesh filename=./meshes/DistalPhalang.dae
- link arm3_link1: geometry collision cylinder length=0.15 radius=0.01; visual mesh filename=./meshes/ProximalPhalang.dae
- link arm3_link2: geometry collision cylinder length=0.25 radius=0.01; visual mesh filename=./meshes/MiddlePhalang.dae
- link arm3_link3: geometry collision cylinder length=0.25 radius=0.01; visual mesh filename=./meshes/DistalPhalang.dae
- link base: geometry collision box size=0.25 0.25 0.05; visual mesh filename=./meshes/FeelyDroneBase.dae

File: feely_drone_common/assets/gripper.xacro (robot description, xacro)
@@ -6,10 +6,13 @@
     <xacro:property name="m_base" value="1.0" />
     <xacro:property name="base_width" value="0.25" />
-    <xacro:property name="depth" value="0.25" />
-    <xacro:property name="height" value="0.05" />
+    <xacro:property name="base_depth" value="0.225" />
+    <xacro:property name="base_height" value="0.08" />
+    <xacro:property name="stack_height" value="0.08" />
+    <xacro:property name="stack_width" value="0.075" />
+    <xacro:property name="stack_depth" value="0.1" />
     <!-- Create three instances of the robot, rotated to form a gripper -->
-    <xacro:r3_robot prefix="arm1" xyz="-${base_width/2} ${depth/2} 0" rpy="${-pi2} 0 0" />
-    <xacro:r3_robot prefix="arm2" xyz=" 0.0       -${depth/2} 0" rpy="${-pi2} 0 ${pi}" />
-    <xacro:r3_robot prefix="arm3" xyz=" ${base_width/2} ${depth/2} 0" rpy="${-pi2} 0 0" />
+    <xacro:r3_robot prefix="arm1" xyz="${-stack_width/2 + 0.014} ${-stack_depth/2 + 0.0175} ${0.5*(base_height)+stack_height}" rpy="${-pi2} 0 ${pi2}" />
+    <xacro:r3_robot prefix="arm2" xyz="${ stack_width/2 - 0.014}  0.0              ${0.5*(base_height)+stack_height}" rpy="${-pi2} 0 ${-pi2}" />
+    <xacro:r3_robot prefix="arm3" xyz="${-stack_width/2 + 0.014} ${ stack_depth/2 - 0.026} ${0.5*(base_height)+stack_height}" rpy="${-pi2} 0 ${pi2}" />
     <!-- Optionally, add a base link or other structure to connect the arms -->
     <link name="world"/>
@@ -17,14 +20,23 @@
     <link name="p2"/>
     <link name="p3"/>
+    <link name="drone">
+        <collision>
+            <origin xyz="0 0 ${base_height*0.25}" rpy="0 0 0"/>
+            <geometry>
+                <box size="${base_width} ${base_depth} ${0.5*base_height}"/>
+            </geometry>
+        </collision>
+    </link>
     <link name="base">
         <visual>
             <geometry>
-                <box size="${base_width} ${depth} ${height}"/>
+                <!--<box size="${base_width} ${base_depth} ${base_height}"/>-->
+                <mesh filename="./meshes/FeelyDroneBase.dae"/>
             </geometry>
         </visual>
         <collision>
-            <origin xyz="0 0 0" rpy="0 0 0"/>
+            <origin xyz="0 0 ${base_height}" rpy="0 0 0"/>
             <geometry>
-                <box size="${base_width} ${depth} ${height}"/>
+                <box size="${stack_width} ${stack_depth} ${stack_height}"/>
             </geometry>
         </collision>
@@ -32,11 +44,15 @@
             <origin xyz="0 0 0" rpy="0 0 0"/>
             <mass value="${m_base}" />
-            <inertia ixx="${1.0/12.0 * m_base * (height*height + depth*depth)}"
+            <inertia ixx="${1.0/12.0 * m_base * (base_height*base_height + base_depth*base_depth)}"
                      ixy="0.0" ixz="0.0"
-                     iyy="${1.0/12.0 * m_base * (height*height + base_width*base_width)}"
+                     iyy="${1.0/12.0 * m_base * (base_height*base_height + base_width*base_width)}"
                      iyz="0.0"
-                     izz="${1.0/12.0 * m_base * (base_width*base_width + depth*depth)}" />
+                     izz="${1.0/12.0 * m_base * (base_width*base_width + base_depth*base_depth)}" />
         </inertial>
     </link>
+    <joint name="droneFixture" type="fixed">
+        <parent link="drone"/>
+        <child link="base"/>
+    </joint>
     <joint name="x_pos" type="prismatic">
         <parent link="world" />

File: feely_drone_common/assets/r3_robot.xacro (robot description, xacro)
@@ -3,7 +3,7 @@
     <xacro:property name="pi2" value="${pi * 0.5}" />
     <xacro:property name="width" value="0.01" />
-    <xacro:property name="l1" value="0.15" />
-    <xacro:property name="l2" value="0.25" />
-    <xacro:property name="l3" value="0.25" />
+    <xacro:property name="l1" value="0.055" />
+    <xacro:property name="l2" value="0.04" />
+    <xacro:property name="l3" value="0.045" />
     <xacro:property name="m1" value="1" />
     <xacro:property name="m2" value="1" />
@@ -14,7 +14,8 @@
         <link name="${prefix}_link1">
             <visual>
-                <origin xyz="0 0 ${l1 * 0.5}" rpy="0 0 0"/>
+                <origin xyz="${-width * 0.5} ${0.0} ${l1 * 0.5}" rpy="0 ${pi2} 0"/>
                 <geometry>
-                    <cylinder radius="${width}" length="${l1}"/>
+                    <mesh filename="./meshes/ProximalPhalang.dae"/>
+                    <!--<cylinder radius="${width}" length="${l1}"/>-->
                 </geometry>
             </visual>
@@ -37,7 +38,7 @@
         <link name="${prefix}_link2">
             <visual>
-                <origin xyz="0 0 ${l2 * 0.5}" rpy="0 0 0"/>
+                <origin xyz="${-width * 0.7} 0 ${l2 * 0.5}" rpy="0 ${pi2} 0"/>
                 <geometry>
-                    <cylinder radius="${width}" length="${l2}"/>
+                    <mesh filename="./meshes/MiddlePhalang.dae"/>
                 </geometry>
             </visual>
@@ -60,7 +61,7 @@
         <link name="${prefix}_link3">
             <visual>
-                <origin xyz="0 0 ${l3 * 0.5}" rpy="0 0 0"/>
+                <origin xyz="0.0026 -0.0082 ${l3 * 0.25}" rpy="0 ${pi2} ${pi2}"/>
                 <geometry>
-                    <cylinder radius="${width}" length="${l3}"/>
+                    <mesh filename="./meshes/DistalPhalang.dae"/>
                 </geometry>
             </visual>
