Commit message: Fix alignment for gripper vis with pads

File: feely_drone_common/assets/r3_robot.xacro (robot description, xacro)
@@ -38,5 +38,5 @@
         <link name="${prefix}_link2">
             <visual>
-                <origin xyz="${-width * 0.7} 0 ${l2 * 0.5}" rpy="0 ${pi2} 0"/>
+                <origin xyz="${width * 0.4} 0 ${l2 * 0.5}" rpy="0 ${pi2} 0"/>
                 <geometry>
                     <mesh filename="./meshes/MiddlePhalang.dae"/>
@@ -61,5 +61,5 @@
         <link name="${prefix}_link3">
             <visual>
-                <origin xyz="0.0026 -0.0082 ${l3 * 0.25}" rpy="0 ${pi2} ${pi2}"/>
+                <origin xyz="-0.0026 0.0082 ${l3 * 0.25}" rpy="0 ${pi2} ${-pi2}"/>
                 <geometry>
                     <mesh filename="./meshes/DistalPhalang.dae"/>
