Commit message: Unify state machine for ros2 and genesis use+add more assests

File: feely_drone_common/assets/cylinder.urdf (robot description, URDF)
Before this commit: robot cylinder, 2 links, 1 joints
Links:
- link base: geometry collision cylinder length=7.07106781185 radius=0.05; visual cylinder length=7.07106781185 radius=0.05

File: feely_drone_common/assets/cylinder.xacro (robot description, xacro)
@@ -2,5 +2,5 @@
 <robot xmlns:xacro="http://www.ros.org/wiki/xacro" name="cylinder">
     <xacro:property name="sqrt2" value="1.41421356237" />
-    <xacro:property name="radius" value="0.125" />
+    <xacro:property name="radius" value="0.05" />
     <xacro:property name="length" value="${5 * sqrt2}" />
     <xacro:property name="m" value="1" />

File: feely_drone_common/assets/gripper.urdf (robot description, URDF)
Before this commit: robot gripper, 17 links, 16 joints
Links:
- added link drone; collision box size=0.25 0.225 0.04
- link arm1_link1: mass 1 -> 0.1; geometry collision cylinder length=0.055 radius=0.01; visual mesh filename=./meshes/ProximalPhalang.dae
- link arm1_link2: mass 1 -> 0.1; geometry collision cylinder length=0.04 radius=0.01; visual mesh filename=./meshes/MiddlePhalang.dae
- link arm1_link3: mass 1 -> 0.1; geometry collision cylinder length=0.045 radius=0.01; visual mesh filename=./meshes/DistalPhalang.dae
- link arm2_link1: mass 1 -> 0.1; geometry collision cylinder length=0.055 radius=0.01; visual mesh filename=./meshes/ProximalPhalang.dae
- link arm2_link2: mass 1 -> 0.1; geometry collision cylinder length=0.04 radius=0.01; visual mesh filename=./meshes/MiddlePhalang.dae
- link arm2_link3: mass 1 -> 0.1; geometry collision cylinder length=0.045 radius=0.01; visual mesh filename=./meshes/DistalPhalang.dae
- link arm3_link1: mass 1 -> 0.1; geometry collision cylinder length=0.055 radius=0.01; visual mesh filename=./meshes/ProximalPhalang.dae
- link arm3_link2: mass 1 -> 0.1; geometry collision cylinder length=0.04 radius=0.01; visual mesh filename=./meshes/MiddlePhalang.dae
- link arm3_link3: mass 1 -> 0.1; geometry collision cylinder length=0.045 radius=0.01; visual mesh filename=./meshes/DistalPhalang.dae
- link base: geometry collision box size=0.075 0.1 0.08; visual mesh filename=./meshes/FeelyDroneBase.dae
Joints:
- added joint droneFixture: type fixed, parent drone, child base
- joint arm1_joint1: origin xyz=-0.125 0.125 0 rpy=-1.5707963267948966 0 0 -> xyz=-0.0235 -0.0325 0.12 rpy=-1.5707963267948966 0 1.5707963267948966
- joint arm1_joint2: origin xyz=0 0 0.15 rpy=0 0 0 -> xyz=0 0 0.055 rpy=0 0 0
- joint arm1_joint3: origin xyz=0 0 0.25 rpy=0 0 0 -> xyz=0 0 0.04 rpy=0 0 0
- joint arm2_joint1: origin xyz= 0.0       -0.125 0 rpy=-1.5707963267948966 0 3.141592653589793 -> xyz=0.0235  0.0              0.12 rpy=-1.5707963267948966 0 -1.5707963267948966
- joint arm2_joint2: origin xyz=0 0 0.15 rpy=0 0 0 -> xyz=0 0 0.055 rpy=0 0 0
- joint arm2_joint3: origin xyz=0 0 0.25 rpy=0 0 0 -> xyz=0 0 0.04 rpy=0 0 0
- joint arm3_joint1: origin xyz= 0.125 0.125 0 rpy=-1.5707963267948966 0 0 -> xyz=-0.0235 0.024000000000000004 0.12 rpy=-1.5707963267948966 0 1.5707963267948966
- joint arm3_joint2: origin xyz=0 0 0.15 rpy=0 0 0 -> xyz=0 0 0.055 rpy=0 0 0
- joint arm3_joint3: origin xyz=0 0 0.25 rpy=0 0 0 -> xyz=0 0 0.04 rpy=0 0 0
- joint base_joint: child base -> drone

File: feely_drone_common/assets/gripper.xacro (robot description, xacro)
@@ -75,5 +75,5 @@
     <joint name="base_joint" type="continuous">
         <parent link="p3" />
-        <child link="base" />
+        <child link="drone" />
         <axis xyz="0 0 1"/>
         <dynamics damping="100.0" friction="0.0"/>

File: feely_drone_common/assets/r3_robot.xacro (robot description, xacro)
@@ -6,7 +6,7 @@
     <xacro:property name="l2" value="0.04" />
     <xacro:property name="l3" value="0.045" />
-    <xacro:property name="m1" value="1" />
-    <xacro:property name="m2" value="1" />
-    <xacro:property name="m3" value="1" />
+    <xacro:property name="m1" value="0.1" />
+    <xacro:property name="m2" value="0.1" />
+    <xacro:property name="m3" value="0.1" />
     <!-- Wrap the entire robot definition in a macro -->
     <xacro:macro name="r3_robot" params="prefix xyz rpy">

Commit message: Make a simple and full mesh vis of the gripper drone
This is exportable via xacro flag full_visuals

File: feely_drone_common/assets/cylinder.urdf (robot description, URDF)
Before this commit: robot cylinder, 2 links, 1 joints
Links:
- link base: geometry collision cylinder length=7.07106781185 radius=0.025; visual cylinder length=7.07106781185 radius=0.025

File: feely_drone_common/assets/cylinder.xacro (robot description, xacro)
@@ -2,5 +2,5 @@
 <robot xmlns:xacro="http://www.ros.org/wiki/xacro" name="cylinder">
     <xacro:property name="sqrt2" value="1.41421356237" />
-    <xacro:property name="radius" value="0.05" />
+    <xacro:property name="radius" value="0.025" />
     <xacro:property name="length" value="${5 * sqrt2}" />
     <xacro:property name="m" value="1" />

File: feely_drone_common/assets/gripper.xacro (robot description, xacro)
@@ -1,4 +1,5 @@
 <?xml version="1.0"?>
 <robot xmlns:xacro="http://www.ros.org/wiki/xacro" name="gripper">
+    <xacro:arg name="full_visuals" default="true"/>
     <!-- Include the robot macro -->
     <xacro:include filename="r3_robot.xacro"/>
@@ -31,6 +32,10 @@
         <visual>
             <geometry>
-                <!--<box size="${base_width} ${base_depth} ${base_height}"/>-->
-                <mesh filename="./meshes/FeelyDroneBase.dae"/>
+                <xacro:if value="$(arg full_visuals)">
+                    <mesh filename="./meshes/FeelyDroneBase.dae"/>
+                </xacro:if>
+                <xacro:unless value="$(arg full_visuals)">
+                    <box size="${base_width} ${base_depth} ${base_height}"/>
+                </xacro:unless>
             </geometry>
         </visual>
@@ -56,4 +61,5 @@
     </joint>
     <joint name="x_pos" type="prismatic">
+        <origin xyz="0 0 ${-base_height-stack_height}" rpy="0 0 0"/>
         <parent link="world" />
         <child link="p1" />

File: feely_drone_common/assets/gripper_simple.urdf (robot description, URDF)
Before this commit: robot gripper, 18 links, 17 joints
Links:
- link arm1_link1: geometry collision cylinder length=0.055 radius=0.01; visual cylinder length=0.055 radius=0.01
- link arm1_link2: geometry collision cylinder length=0.04 radius=0.01; visual cylinder length=0.04 radius=0.01
- link arm1_link3: geometry collision cylinder length=0.045 radius=0.01; visual cylinder length=0.045 radius=0.01
- link arm2_link1: geometry collision cylinder length=0.055 radius=0.01; visual cylinder length=0.055 radius=0.01
- link arm2_link2: geometry collision cylinder length=0.04 radius=0.01; visual cylinder length=0.04 radius=0.01
- link arm2_link3: geometry collision cylinder length=0.045 radius=0.01; visual cylinder length=0.045 radius=0.01
- link arm3_link1: geometry collision cylinder length=0.055 radius=0.01; visual cylinder length=0.055 radius=0.01
- link arm3_link2: geometry collision cylinder length=0.04 radius=0.01; visual cylinder length=0.04 radius=0.01
- link arm3_link3: geometry collision cylinder length=0.045 radius=0.01; visual cylinder length=0.045 radius=0.01
- link base: geometry collision box size=0.075 0.1 0.08; visual box size=0.25 0.225 0.08

File: feely_drone_common/assets/r3_robot.xacro (robot description, xacro)
@@ -14,9 +14,16 @@
         <link name="${prefix}_link1">
             <visual>
-                <origin xyz="${-width * 0.5} ${0.0} ${l1 * 0.5}" rpy="0 ${pi2} 0"/>
-                <geometry>
-                    <mesh filename="./meshes/ProximalPhalang.dae"/>
-                    <!--<cylinder radius="${width}" length="${l1}"/>-->
-                </geometry>
+                <xacro:if value="$(arg full_visuals)">
+                    <origin xyz="${-width * 0.5} ${0.0} ${l1 * 0.5}" rpy="0 ${pi2} 0"/>
+                    <geometry>
+                        <mesh filename="./meshes/ProximalPhalang.dae"/>
+                    </geometry>
+                </xacro:if>
+                <xacro:unless value="$(arg full_visuals)">
+                    <origin xyz="0 0 ${l1 * 0.5}" rpy="0 0 0"/>
+                    <geometry>
+                        <cylinder radius="${width}" length="${l1}"/>
+                    </geometry>
+                </xacro:unless>
             </visual>
             <collision>
@@ -38,8 +45,16 @@
         <link name="${prefix}_link2">
             <visual>
-                <origin xyz="${width * 0.4} 0 ${l2 * 0.5}" rpy="0 ${pi2} 0"/>
-                <geometry>
-                    <mesh filename="./meshes/MiddlePhalang.dae"/>
-                </geometry>
+                <xacro:if value="$(arg full_visuals)">
+                    <origin xyz="${width * 0.4} 0 ${l2 * 0.5}" rpy="0 ${pi2} 0"/>
+                    <geometry>
+                        <mesh filename="./meshes/MiddlePhalang.dae"/>
+                    </geometry>
+                </xacro:if>
+                <xacro:unless value="$(arg full_visuals)">
+                    <origin xyz="0 0 ${l2 * 0.5}" rpy="0 0 0"/>
+                    <geometry>
+                        <cylinder radius="${width}" length="${l2}"/>
+                    </geometry>
+                </xacro:unless>
             </visual>
             <collision>
@@ -61,8 +76,16 @@
         <link name="${prefix}_link3">
             <visual>
-                <origin xyz="-0.0026 0.0082 ${l3 * 0.25}" rpy="0 ${pi2} ${-pi2}"/>
-                <geometry>
-                    <mesh filename="./meshes/DistalPhalang.dae"/>
-                </geometry>
+                <xacro:if value="$(arg full_visuals)">
+                    <origin xyz="-0.0026 0.0082 ${l3 * 0.25}" rpy="0 ${pi2} ${-pi2}"/>
+                    <geometry>
+                        <mesh filename="./meshes/DistalPhalang.dae"/>
+                    </geometry>
+                </xacro:if>
+                <xacro:unless value="$(arg full_visuals)">
+                    <origin xyz="0 0 ${l3 * 0.5}" rpy="0 0 0"/>
+                    <geometry>
+                        <cylinder radius="${width}" length="${l3}"/>
+                    </geometry>
+                </xacro:unless>
             </visual>
             <collision>

Commit message: Fine tune assets

File: feely_drone_common/assets/cylinder.urdf (robot description, URDF)
Before this commit: robot cylinder, 2 links, 1 joints
Links:
- link base: geometry collision cylinder length=7.07106781185 radius=0.03; visual cylinder length=7.07106781185 radius=0.03

File: feely_drone_common/assets/cylinder.xacro (robot description, xacro)
@@ -2,5 +2,5 @@
 <robot xmlns:xacro="http://www.ros.org/wiki/xacro" name="cylinder">
     <xacro:property name="sqrt2" value="1.41421356237" />
-    <xacro:property name="radius" value="0.025" />
+    <xacro:property name="radius" value="0.03" />
     <xacro:property name="length" value="${5 * sqrt2}" />
     <xacro:property name="m" value="1" />

File: feely_drone_common/assets/gripper.urdf (robot description, URDF)
Before this commit: robot gripper, 18 links, 17 joints
Joints:
- joint x_pos: origin xyz=0 0 -0.16 rpy=0 0 0 -> xyz=0 0 -0.08 rpy=0 0 0

File: feely_drone_common/assets/gripper.xacro (robot description, xacro)
@@ -61,5 +61,5 @@
     </joint>
     <joint name="x_pos" type="prismatic">
-        <origin xyz="0 0 ${-base_height-stack_height}" rpy="0 0 0"/>
+        <origin xyz="0 0 ${-stack_height}" rpy="0 0 0"/>
         <parent link="world" />
         <child link="p1" />

File: feely_drone_common/assets/gripper_simple.urdf (robot description, URDF)
Before this commit: robot gripper, 18 links, 17 joints
Joints:
- joint x_pos: origin xyz=0 0 -0.16 rpy=0 0 0 -> xyz=0 0 -0.08 rpy=0 0 0
