Commit message: Fix cylinder orientation

File: feely_drone_common/assets/cylinder.xacro (robot description, xacro)
@@ -10,5 +10,5 @@
         <link name="base">
             <visual>
-                <origin xyz="0 0 0" rpy="0 0 0"/>
+                <origin xyz="0 0 0" rpy="1.57079633 0 0"/>
                 <geometry>
                     <cylinder radius="${radius}" length="${length}"/>
@@ -16,5 +16,5 @@
             </visual>
             <collision>
-                <origin xyz="0 0 0" rpy="0 0 0"/>
+                <origin xyz="0 0 0" rpy="1.57079633 0 0"/>
                 <geometry>
                     <cylinder radius="${radius}" length="${length}"/>

Commit message: make many cylinders urdf

File: feely_drone_common/assets/cylinder.xacro (robot description, xacro)
@@ -2,7 +2,10 @@
 <robot xmlns:xacro="http://www.ros.org/wiki/xacro" name="cylinder">
     <xacro:property name="sqrt2" value="1.41421356237" />
-    <xacro:property name="radius" value="0.03" />
+    <xacro:arg name="base_path" default="./"/>
+    <xacro:arg name="cylinder_radius" default="0.03"/>
+    <xacro:property name="radius" value="$(arg cylinder_radius)"/>
     <xacro:property name="length" value="${5 * sqrt2}" />
     <xacro:property name="m" value="1" />
+    <xacro:arg name="full_visuals" default="true"/>
     <!-- Wrap the entire robot definition in a macro -->
     <xacro:macro name="cylinder" params="xyz rpy">
@@ -14,4 +17,10 @@
                     <cylinder radius="${radius}" length="${length}"/>
                 </geometry>
+                <xacro:if value="$(arg full_visuals)">
+                    <material name="cylinder_material">
+                        <color rgba="1.0 1.0 1.0 1.0"/>
+                        <texture filename="$(arg base_path)textures/tree_bark.jpg"/>
+                    </material>
+                </xacro:if>
             </visual>
             <collision>

File: feely_drone_common/assets/cylinders/cylinder_0.425.urdf (robot description, URDF)
Before this commit: robot cylinder, 2 links, 1 joints
Links:
- link base: geometry collision cylinder length=7.07106781185 radius=0.425; visual cylinder length=7.07106781185 radius=0.425
