Commit message: Add hbars to assets

File: feely_drone_common/assets/cyberzoo.urdf (robot description, URDF)
Before this commit: robot cyberzoo, 1 links, 0 joints
Links:
- link cyberzoo_link: geometry visual mesh filename=meshes/cyberzoo/cyberzoo_cams.dae; visual mesh filename=meshes/cyberzoo/cyberzoo_floor.dae
